File: Drivetrain_schematic.kicad_sch (KiCad schematic)
At the start: 4 parts

Commit message: schematic
Parts:
- added 9V: (no value), symbol Device:Battery
- renumbered motor_driver to H-bridge_driver
Connections:
- net motor_driver_5V is gone; now on net 5V: microcontroller.5 (+5V)
- net GND: now also 9V.2 (-)
- net arduino 5V renamed 5V
- net battery +: no longer names the net of H-bridge_driver.9 (+12V)
- net battery +: now also 9V.1 (+)
Other:
- moved on the sheet: microcontroller
